File: pcb/lemmingz40/lemmingz40.kicad_pcb (KiCad board)
At the start: 2 copper layers, 115.4 x 48.1 mm, 107 parts, among them J1 USB_C_Receptacle_USB2.0, SW1 SW_Push, SW10 SW_Push, SW11 SW_Push, SW12 SW_Push, SW13 SW_Push, SW14 SW_Push, SW15 SW_Push, SW16 SW_Push, SW17 SW_Push, SW18 SW_Push, SW19 SW_Push, SW2 SW_Push, SW20 SW_Push, SW21 SW_Push, SW22 SW_Push, SW23 SW_Push, SW24 SW_Push, SW25 SW_Push, SW26 SW_Push, SW27 SW_Push, SW28 SW_Push, SW29 SW_Push, SW3 SW_Push, SW30 SW_Push, SW31 SW_Push, SW32 SW_Push, SW33 SW_Push, SW34 SW_Push, SW35 SW_Push, SW36 SW_Push, SW37 SW_Push, SW38 SW_Push, SW39 SW_Push, SW4 SW_Push, SW40 SW_Push, SW41 RST, SW42 RST, SW5 SW_Push, SW6 SW_Push, SW7 SW_Push, SW8 SW_Push, SW9 SW_Push, U1 USBLC6-2SC6, U2 STM32F072C8Tx, U3 XC6206PxxxMR-Regulator_Linear

Commit message: add v0.0 exports
Parts:
- H1, H2, H3, H4, H5, H6, H7, H8: value MountingHole -> MountingHole_Pad; footprint userlib:m1.6_hole -> userlib:SMTSO-M1.6; moved to B.Cu
- J1: value USB_C_Receptacle_USB2.0 -> USB2_C_Receptacle; footprint Connector_USB:USB_C_Receptacle_XKB_U262-16XN-4BVC11 -> userlib:Mid_Mount-USB_C
- SW41: value RST -> BOOT
- moved H3 27.4 mm to (46.1, 66.1), turned to 170 degrees
- moved H1 21.3 mm to (49.6, 46.3), turned to 170 degrees
- moved J1 3.58 mm to (92.7, 34.8), turned to 90 degrees
- moved H2 1.50 mm to (79.2, 51.5), turned to 170 degrees
- moved SW20 1.43 mm to (102.2, 57.4)
- moved SW23 1.43 mm to (51.9, 62.0)
- moved D18 1.43 mm to (116.2, 56.4)
- moved SW12 1.43 mm to (141.6, 50.4)
- moved C6 1.43 mm to (86.5, 68.0)
- moved D6 1.43 mm to (124.4, 44.8)
- moved C2 1.43 mm to (92.6, 58.9)
- moved SW1 1.43 mm to (45.5, 40.6)
- moved SW19 1.43 mm to (83.2, 57.4)
- moved SW4 1.43 mm to (130.0, 42.3)
- moved SW13 1.43 mm to (53.6, 52.2)
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Connections:
- H1 pad 1: (no net) -> GND
- H2 pad 1: (no net) -> GND
- H3 pad 1: (no net) -> GND
- H4 pad 1: (no net) -> GND
- H5 pad 1: (no net) -> GND
- H6 pad 1: (no net) -> GND
- H7 pad 1: (no net) -> GND
- H8 pad 1: (no net) -> GND
- J1 pad A6: D_USB_+ -> D_USB_-
- J1 pad A7: D_USB_- -> D_USB_+
- J1 pad B6: D_USB_+ -> D_USB_-
- J1 pad B7: D_USB_- -> D_USB_+
- U2 pad 15: COL10 -> unconnected-(U2-PA5-Pad15)
- U2 pad 16: COL9 -> unconnected-(U2-PA6-Pad16)
- U2 pad 17: COL8 -> unconnected-(U2-PA7-Pad17)
- U2 pad 18: COL6 -> COL9
- U2 pad 19: unconnected-(U2-PB1-Pad19) -> COL7
- U2 pad 2: unconnected-(U2-PC13-Pad2) -> COL2
- U2 pad 20: unconnected-(U2-PB2-Pad20) -> COL5
- U2 pad 21: ROW3 -> COL3
- U2 pad 22: ROW2 -> COL1
- U2 pad 25: COL5 -> unconnected-(U2-PB12-Pad25)
- U2 pad 26: COL4 -> unconnected-(U2-PB13-Pad26)
- U2 pad 27: COL3 -> ROW4
- U2 pad 28: COL2 -> ROW3
- U2 pad 29: COL1 -> ROW2
- U2 pad 3: unconnected-(U2-PC14-Pad3) -> COL4
- U2 pad 30: COL0 -> ROW1
- U2 pad 37: ROW1 -> unconnected-(U2-PA14-Pad37)
- U2 pad 38: ROW0 -> unconnected-(U2-PA15-Pad38)
- U2 pad 39: COL7 -> unconnected-(U2-PB3-Pad39)
- U2 pad 4: unconnected-(U2-PC15-Pad4) -> COL6
- U2 pad 40: LED_SLCK -> unconnected-(U2-PB4-Pad40)
- U2 pad 5: unconnected-(U2-PF0-Pad5) -> COL8
- U2 pad 6: unconnected-(U2-PF1-Pad6) -> COL10
Routing:
- net GND: track 111.2 -> 344.6 mm, vias 4 -> 6
- net COL2: track 210.0 -> 272.2 mm, vias 0 -> 2
- net COL1: track 210.0 -> 270.5 mm, vias 0 -> 2
- net COL4: track 210.0 -> 262.7 mm, vias 0 -> 2
- net COL3: track 210.0 -> 260.3 mm, vias 0 -> 2
- net ROW3: track 120.0 -> 166.5 mm, vias 0 -> 2
- net ROW4: track 122.0 -> 167.6 mm, vias 0 -> 3
- net COL6: track 210.0 -> 244.7 mm
- net COL5: track 210.0 -> 240.2 mm, vias 0 -> 1
- net ROW2: track 100.0 -> 125.6 mm, vias 0 -> 2
- net COL8: track 210.0 -> 234.5 mm
- net COL7: track 210.0 -> 229.2 mm, vias 0 -> 1
- net COL10: track 210.0 -> 227.4 mm
- net COL9: track 210.0 -> 222.2 mm, vias 0 -> 2
- net VBUS: track 36.1 -> 24.4 mm, vias 5 -> 4
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Other:
- outline, holes or cut-outs redrawn
- board text added: "boot"
- board text added: "lemmingz40 v0.0 by sporewoh"
- board text added: "reset"
- board text added: "科学は行き過ぎてしまった のでしょうか？？"

Commit message: add exports and photos
Connections:
- U1 pad 5: VBUS -> +5V
Routing:
- net +5V: track 9.42 -> 19.9 mm, vias 2 -> 4
- net GND: track 344.6 -> 351.2 mm, vias 6 -> 8
- net VBUS: track 24.4 -> 22.5 mm, vias 4 -> 3

Commit message: update serial wire error, make standoffs 2mm from 1.5mm
Connections:
- J1 pad A6: D_USB_- -> D_USB_+
- J1 pad A7: D_USB_+ -> D_USB_-
- J1 pad B6: D_USB_- -> D_USB_+
- J1 pad B7: D_USB_+ -> D_USB_-
Routing:
- net D_USB_-: track 7.43 -> 6.55 mm, vias 2 -> 0
Other:
- board text added: "lemmingz40 v0.1 by sporewoh"
- board text removed: "lemmingz40 v0.0 by sporewoh"
Changed lines of the file:
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@@
       (net 50 "Net-(J1-CC1)") (pinfunction "CC1") (pintype "passive"))
     (pad "A6" smd rect (at -7.63 -0.25) (size 0.3 1.1) (layers "B.Cu" "B.Paste" "B.Mask")
-      (net 52 "D_USB_-") (pinfunction "D+") (pintype "passive"))
+      (net 51 "D_USB_+") (pinfunction "D+") (pintype "passive"))
     (pad "A7" smd rect (at -7.63 0.25) (size 0.3 1.1) (layers "B.Cu" "B.Paste" "B.Mask")
-      (net 51 "D_USB_+") (pinfunction "D-") (pintype "passive"))
+      (net 52 "D_USB_-") (pinfunction "D-") (pintype "passive"))
     (pad "A8" smd rect (at -7.63 1.25) (size 0.3 1.1) (layers "B.Cu" "B.Paste" "B.Mask")
       (net 53 "unconnected-(J1-SBU1-PadA8)") (pinfunction "SBU1") (pintype "passive+no_connect"))
@@
       (net 54 "Net-(J1-CC2)") (pinfunction "CC2") (pintype "passive"))
     (pad "B6" smd rect (at -7.63 0.75) (size 0.3 1.1) (layers "B.Cu" "B.Paste" "B.Mask")
-      (net 52 "D_USB_-") (pinfunction "D+") (pintype "passive"))
+      (net 51 "D_USB_+") (pinfunction "D+") (pintype "passive"))
     (pad "B7" smd rect (at -7.63 -0.75) (size 0.3 1.1) (layers "B.Cu" "B.Paste" "B.Mask")
-      (net 51 "D_USB_+") (pinfunction "D-") (pintype "passive"))
+      (net 52 "D_USB_-") (pinfunction "D-") (pintype "passive"))
     (pad "B8" smd rect (at -7.63 -1.75) (size 0.3 1.1) (layers "B.Cu" "B.Paste" "B.Mask")
       (net 55 "unconnected-(J1-SBU2-PadB8)") (pinfunction "SBU2") (pintype "passive+no_connect"))
@@
     (effects (font (size 1 1) (thickness 0.1)) (justify left bottom mirror))
   )
-  (gr_text "lemmingz40\nv0.0\nby sporewoh" (at 113.333288 39.999984) (layer "B.SilkS")
+  (gr_text "lemmingz40\nv0.1\nby sporewoh" (at 113.333288 39.999984) (layer "B.SilkS")
     (effects (font (size 1 1) (thickness 0.25) bold) (justify bottom mirror))
   )
@@
   (segment (start 91.360049 44.575352) (end 91.410012 44.525388) (width 0.25) (layer "B.Cu") (net 50))
   (segment (start 89.003345 44.418649) (end 89.060048 44.475351) (width 0.25) (layer "B.Cu") (net 50))
-  (segment (start 92.910012 41.670012) (end 92.910012 42.384151) (width 0.2) (layer "B.Cu") (net 51))
-  (segment (start 92.885011 44.885745) (end 92.885012 42.061063) (width 0.2) (layer "B.Cu") (net 51))
-  (segment (start 92.774151 41.534151) (end 92.910012 41.670012) (width 0.2) (layer "B.Cu") (net 51))
-  (segment (start 93.610012 46.604498) (end 93.610014 45.610748) (width 0.2) (layer "B.Cu") (net 51))
-  (segment (start 91.910012 42.384151) (end 91.910012 41.759887) (width 0.2) (layer "B.Cu") (net 51))
-  (segment (start 91.910012 41.759887) (end 92.135748 41.534151) (width 0.2) (layer "B.Cu") (net 51))
-  (segment (start 92.135748 41.534151) (end 92.774151 41.534151) (width 0.2) (layer "B.Cu") (net 51))
-  (segment (start 93.610014 45.610748) (end 92.885011 44.885745) (width 0.2) (layer "B.Cu") (net 51))
-  (segment (start 93.544839 43.520328) (end 93.584511 43.56) (width 0.2) (layer "F.Cu") (net 52))
-  (segment (start 92.185704 43.520328) (end 93.544839 43.520328) (width 0.2) (layer "F.Cu") (net 52))
-  (via (at 93.584511 43.56) (size 0.8) (drill 0.4) (layers "F.Cu" "B.Cu") (net 52))
-  (via (at 92.185704 43.520328) (size 0.8) (drill 0.4) (layers "F.Cu" "B.Cu") (net 52))
-  (segment (start 92.410012 44.860748) (end 92.435011 44.885747) (width 0.2) (layer "B.Cu") (net 52))
-  (segment (start 92.206032 43.5) (end 92.185704 43.520328) (width 0.2) (layer "B.Cu") (net 52))
-  (segment (start 93.410012 43.385501) (end 93.410012 42.384151) (width 0.2) (layer "B.Cu") (net 52))
-  (segment (start 93.584511 43.56) (end 93.410012 43.385501) (width 0.2) (layer "B.Cu") (net 52))
-  (segment (start 91.710012 45.610747) (end 92.435011 44.885747) (width 0.2) (layer "B.Cu") (net 52))
-  (segment (start 91.710012 46.604498) (end 91.710012 45.610747) (width 0.2) (layer "B.Cu") (net 52))
-  (segment (start 92.410012 43.5) (end 92.206032 43.5) (width 0.2) (layer "B.Cu") (net 52))
-  (segment (start 92.410012 42.384151) (end 92.410012 43.5) (width 0.2) (layer "B.Cu") (net 52))
-  (segment (start 92.410012 43.5) (end 92.410012 44.860748) (width 0.2) (layer "B.Cu") (net 52))
+  (segment (start 93.410012 41.743366) (end 93.410012 42.384151) (width 0.2) (layer "B.Cu") (net 51))
+  (segment (start 92.410012 41.759887) (end 92.635748 41.534151) (width 0.2) (layer "B.Cu") (net 51))
+  (segment (start 92.635748 41.534151) (end 93.200797 41.534151) (width 0.2) (layer "B.Cu") (net 51))
+  (segment (start 92.410012 42.384151) (end 92.410012 41.759887) (width 0.2) (layer "B.Cu") (net 51))
+  (segment (start 93.610012 46.241998) (end 93.610012 46.604498) (width 0.2) (layer "B.Cu") (net 51))
+  (segment (start 93.410012 46.404498) (end 93.610012 46.604498) (width 0.2) (layer "B.Cu") (net 51))
+  (segment (start 93.385012 43.234152) (end 93.385012 44.433133) (width 0.2) (layer "B.Cu") (net 51))
+  (segment (start 93.410012 43.209152) (end 93.385012 43.234152) (width 0.2) (layer "B.Cu") (net 51))
+  (segment (start 92.885012 44.933133) (end 92.885012 45.516998) (width 0.2) (layer "B.Cu") (net 51))
+  (segment (start 93.200797 41.534151) (end 93.410012 41.743366) (width 0.2) (layer "B.Cu") (net 51))
+  (segment (start 93.410012 42.384151) (end 93.410012 43.209152) (width 0.2) (layer "B.Cu") (net 51))
+  (segment (start 93.385012 44.433133) (end 92.885012 44.933133) (width 0.2) (layer "B.Cu") (net 51))
+  (segment (start 92.885012 45.516998) (end 93.610012 46.241998) (width 0.2) (layer "B.Cu") (net 51))
+  (segment (start 92.935012 43.234152) (end 92.935012 44.246733) (width 0.2) (layer "B.Cu") (net 52))
+  (segment (start 92.910012 43.209152) (end 92.935012 43.234152) (width 0.2) (layer "B.Cu") (net 52))
+  (segment (start 92.435012 45.516998) (end 91.710012 46.241998) (width 0.2) (layer "B.Cu") (net 52))
+  (segment (start 92.935012 44.246733) (end 92.435012 44.746733) (width 0.2) (layer "B.Cu") (net 52))
+  (segment (start 92.435012 44.746733) (end 92.435012 45.516998) (width 0.2) (layer "B.Cu") (net 52))
+  (segment (start 91.710012 46.241998) (end 91.710012 46.604498) (width 0.2) (layer "B.Cu") (net 52))
+  (segment (start 92.234913 43.333316) (end 92.785848 43.333316) (width 0.2) (layer "B.Cu") (net 52))
+  (segment (start 91.910012 43.008415) (end 92.234913 43.333316) (width 0.2) (layer "B.Cu") (net 52))
+  (segment (start 91.910012 42.384151) (end 91.910012 43.008415) (width 0.2) (layer "B.Cu") (net 52))
+  (segment (start 92.785848 43.333316) (end 92.910012 43.209152) (width 0.2) (layer "B.Cu") (net 52))
+  (segment (start 92.910012 43.209152) (end 92.910012 42.384151) (width 0.2) (layer "B.Cu") (net 52))
   (segment (start 95.408662 44.575349) (end 95.833295 44.999982) (width 0.25) (layer "F.Cu") (net 54))
   (segment (start 94.185512 44.575349) (end 95.408662 44.575349) (width 0.25) (layer "F.Cu") (net 54))

Commit message: update silkscreen
Other:
- board text added: "modkipz40 v0.1 by sporewoh"
- board text removed: "lemmingz40 v0.1 by sporewoh"
Changed lines of the file:
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@@
     (effects (font (size 1 1) (thickness 0.1)) (justify left bottom mirror))
   )
-  (gr_text "lemmingz40\nv0.1\nby sporewoh" (at 113.333288 39.999984) (layer "B.SilkS")
+  (gr_text "modkipz40\nv0.1\nby sporewoh" (at 113.333288 39.999984) (layer "B.SilkS")
     (effects (font (size 1 1) (thickness 0.25) bold) (justify bottom mirror))
   )
